File: kicad/k1-aioc/k1-aioc.kicad_sch (KiCad schematic)
At the start: 66 parts, among them J1 12401832E402A, J2 Conn_01x07_Male, J3 FT817-CAT, J4 FT817-CAT, Q1 BC847BS, Q2 BC847BS, U1 MIC5330-SSYML, U2 STM32F373CBTx, Y1 8MHz/20pF

Commit message: Board mostly done. Added 817 connectors
Parts:
- removed J2: Conn_01x07_Male, Connector_PinHeader_1.27mm:PinHeader_1x07_P1.27mm_Vertical, symbol Connector:Conn_01x07_Male
- removed Q1, Q2: BC847BS, Package_TO_SOT_SMD:SOT-363_SC-70-6, symbol Device:Q_Dual_NPN_NPN_E1B1C2E2B2C1
- added H3, H4: MountingHole_Pad, MountingHole:MountingHole_3.2mm_M3_ISO14580_Pad, symbol Mechanical:MountingHole_Pad
- added J5: USB, Connector_JST:JST_PH_B4B-PH-K_1x04_P2.00mm_Vertical, symbol Connector:Conn_01x04_Pin
- added J6: Conn_ARM_SWD_TagConnect_TC2030-NL, Connector:Tag-Connect_TC2030-IDC-NL_2x03_P1.27mm_Vertical, symbol Connector:Conn_ARM_SWD_TagConnect_TC2030-NL
- added JP1: SolderJumper_2_Open, Jumper:SolderJumper-2_P1.3mm_Open_TrianglePad1.0x1.5mm, symbol Jumper:SolderJumper_2_Open
- added Q1, Q3, Q4: MMBT3904, Package_TO_SOT_SMD:SOT-23, symbol Transistor_BJT:MMBT3904
- C1, C2: footprint Capacitor_SMD:C_0603_1608Metric -> Capacitor_SMD:C_0402_1005Metric; LCSC C1653 -> C1555
- C11: footprint Capacitor_SMD:C_0603_1608Metric -> Capacitor_SMD:C_0402_1005Metric; LCSC C57112 -> C15195
- C12, C15, C3, C8, C9: footprint Capacitor_SMD:C_0603_1608Metric -> Capacitor_SMD:C_0402_1005Metric; LCSC C14663 -> C307331
- J3: footprint Connector_PinHeader_2.54mm:PinHeader_1x04_P2.54mm_Vertical -> Connector_JST:JST_PH_B3B-PH-K_1x03_P2.00mm_Vertical; symbol Connector:Conn_01x04_Pin -> Connector:Conn_01x03_Pin
- J4: footprint Connector_PinHeader_2.54mm:PinHeader_1x04_P2.54mm_Vertical -> Connector_JST:JST_PH_B4B-PH-K_1x04_P2.00mm_Vertical
- R1: footprint Resistor_SMD:R_0603_1608Metric -> Resistor_SMD:R_0402_1005Metric; LCSC C22843 -> C25867
- R10, R11, R14, R20, R5: footprint Resistor_SMD:R_0603_1608Metric -> Resistor_SMD:R_0402_1005Metric; LCSC C4190 -> C25879
- R12, R13, R18, R21, R22, R23: footprint Resistor_SMD:R_0603_1608Metric -> Resistor_SMD:R_0402_1005Metric; LCSC C23345 -> C25092
- R15, R4, R8, R9: footprint Resistor_SMD:R_0603_1608Metric -> Resistor_SMD:R_0402_1005Metric; LCSC C22962 -> C25091
- R16, R3, R6, R7: footprint Resistor_SMD:R_0603_1608Metric -> Resistor_SMD:R_0402_1005Metric; LCSC C23186 -> C25905
- R17: value N.M. -> DNP; footprint Resistor_SMD:R_0603_1608Metric -> Resistor_SMD:R_0402_1005Metric
- R19: footprint Resistor_SMD:R_0603_1608Metric -> Resistor_SMD:R_0402_1005Metric
- R2: footprint Resistor_SMD:R_0603_1608Metric -> Resistor_SMD:R_0402_1005Metric; LCSC C25804 -> C25744
Connections:
- net +3V3: now also J6.1 (VCC), JP1.1 (A)
- net BOOT0: now also JP1.2 (B)
- net GND: now also J3.3 (Pin_3), H3.1, H4.1, J5.4 (Pin_4), J6.5 (GND), Q1.2 (E), Q3.2 (E), Q4.2 (E); no longer J3.4 (Pin_4)
- net NRST: now also J6.3 (~{RESET})
- net SWCLK: now also J6.4 (SWCLK)
- net SWDIO: now also J6.2 (SWDIO)
- net SWO: now also J6.6 (SWO)
- net USB-DN: now also J5.2 (Pin_2)
- net USB-DP: now also J5.3 (Pin_3)
- net VBUS: now also J5.1 (Pin_1)
- net at R13.2: now also Q3.3 (C)
- net at R11.2: now also Q3.1 (B)
- net at R21.2: now also Q4.3 (C)
- net at R20.1: now also Q4.1 (B)
- net at R12.2: now also Q1.3 (C)
- net at R10.2: now also Q1.1 (B)
Other:
- note removed: "STM Disco SWD Header"

Commit message: Commit before assembly
Parts:
- added H10, H12, H13, H14, H15, H5, H6, H7, H8, H9: Breakaway Hole, AIOC:breakawayHole, symbol Mechanical:MountingHole
- H3, H4: footprint MountingHole:MountingHole_3.2mm_M3_ISO14580_Pad -> MountingHole:MountingHole_2.2mm_M2_ISO14580_Pad_TopBottom
Connections:
- net at R22.1: now also J3.2 (Pin_2); no longer J3.1 (Pin_1)
- net V_SW1_CTRL: now reaches U2.2 (PC13)
- net at R23.1: now also J3.1 (Pin_1); no longer J3.2 (Pin_2)
Other:
- moved on the sheet: R22, R23
