File: kicad/k1-aioc/k1-aioc.kicad_pcb (KiCad board)
At the start: 2 copper layers, 21 x 31.5 mm, 47 parts, among them J1 12401832E402A, J2 Conn_01x07_Male, Q1 BC847BS, U1 MIC5330-SSYML, U2 STM32F373CBTx, Y1 8MHz/20pF

Commit message: Added pin headers for 817
Parts:
- added J3: FT817-CAT, Connector_PinHeader_2.54mm:PinHeader_1x04_P2.54mm_Vertical, F.Cu at (113.5, 119.0)
- added J4: FT817-CAT, Connector_PinHeader_2.54mm:PinHeader_1x04_P2.54mm_Vertical, F.Cu at (117.0, 119.0)
- added Q2: BC847BS, Package_TO_SOT_SMD:SOT-363_SC-70-6, F.Cu at (120.3, 136.2)
- added R18: 22R, Resistor_SMD:R_0603_1608Metric, F.Cu at (119.5, 113.8)
- added R19: DNP, Resistor_SMD:R_0603_1608Metric, F.Cu at (118.0, 114.0)
- added R20: 2.2K, Resistor_SMD:R_0603_1608Metric, F.Cu at (106.9, 128.4)
- added R21: 22R, Resistor_SMD:R_0603_1608Metric, F.Cu at (106.9, 130.9)
- added R22: 22R, Resistor_SMD:R_0603_1608Metric, F.Cu at (106.9, 133.4)
- added R23: 22R, Resistor_SMD:R_0603_1608Metric, F.Cu at (106.9, 135.9)
- added TP1: TestPoint, TestPoint:TestPoint_Pad_1.0x1.0mm, F.Cu at (130.5, 101.5)
- added TP11: TestPoint, TestPoint:TestPoint_Pad_1.0x1.0mm, F.Cu at (125.8, 123.7)
- added TP12: TestPoint, TestPoint:TestPoint_Pad_1.0x1.0mm, F.Cu at (125.8, 126.7)
- added TP13: TestPoint, TestPoint:TestPoint_Pad_1.0x1.0mm, F.Cu at (125.8, 129.8)
- added TP2: TestPoint, TestPoint:TestPoint_Pad_1.0x1.0mm, F.Cu at (119.7, 126.7)
- added TP3: TestPoint, TestPoint:TestPoint_Pad_1.0x1.0mm, F.Cu at (119.7, 129.8)
- added TP4: TestPoint, TestPoint:TestPoint_Pad_1.0x1.0mm, F.Cu at (119.7, 132.8)
- added TP5: TestPoint, TestPoint:TestPoint_Pad_1.0x1.0mm, F.Cu at (122.8, 123.7)
- added TP6: TestPoint, TestPoint:TestPoint_Pad_1.0x1.0mm, F.Cu at (122.8, 126.7)
- added TP7: TestPoint, TestPoint:TestPoint_Pad_1.0x1.0mm, F.Cu at (122.8, 129.8)
- added TP8: TestPoint, TestPoint:TestPoint_Pad_1.0x1.0mm, F.Cu at (122.8, 132.8)
Connections:
- U2 pad 12: unconnected-(U2-Pad12) -> Net-(U2-PA2)
- U2 pad 15: unconnected-(U2-Pad15) -> Net-(U2-PA5)
- U2 pad 16: unconnected-(U2-Pad16) -> Net-(U2-PA6)
- U2 pad 18: unconnected-(U2-Pad18) -> Net-(U2-PB0)
- U2 pad 19: unconnected-(U2-Pad19) -> Net-(U2-PB1)
- U2 pad 26: unconnected-(U2-Pad26) -> Net-(U2-PB14)
- U2 pad 27: unconnected-(U2-Pad27) -> Net-(U2-PB15)
- U2 pad 29: unconnected-(U2-Pad29) -> Net-(U2-PA8)
- U2 pad 38: unconnected-(U2-Pad38) -> Net-(U2-PA15)
- U2 pad 4: unconnected-(U2-Pad4) -> /817_PTT
- U2 pad 40: unconnected-(U2-Pad40) -> Net-(U2-PB4)
- U2 pad 41: unconnected-(U2-Pad41) -> Net-(U2-PB5)
- U2 pad 42: unconnected-(U2-Pad42) -> /817_RX
- U2 pad 43: unconnected-(U2-Pad43) -> /817_TX
Routing:
- net /RADIO-RX-PTT1: track 30.0 -> 37.3 mm
- net Net-(D1-K): track 7.30 -> 9.90 mm
- net Net-(D1-A): track 10.2 -> 12.8 mm
- added copper zone on In1.Cu, net GND
Other:
- copper layers 2 -> 4

Commit message: Board mostly done. Added 817 connectors
Parts:
- removed J2: Conn_01x07_Male, Connector_PinHeader_1.27mm:PinHeader_1x07_P1.27mm_Vertical
- removed Q2: BC847BS, Package_TO_SOT_SMD:SOT-363_SC-70-6
- added H3: MountingHole_Pad, MountingHole:MountingHole_3.2mm_M3_ISO14580_Pad, F.Cu at (121.2, 83.8)
- added H4: MountingHole_Pad, MountingHole:MountingHole_3.2mm_M3_ISO14580_Pad, F.Cu at (106.3, 118.8)
- added J5: USB, Connector_JST:JST_PH_B4B-PH-K_1x04_P2.00mm_Vertical, B.Cu at (114.5, 82.3)
- added J6: Conn_ARM_SWD_TagConnect_TC2030-NL, Connector:Tag-Connect_TC2030-IDC-NL_2x03_P1.27mm_Vertical, B.Cu at (105.7, 86.5)
- added JP1: SolderJumper_2_Open, Jumper:SolderJumper-2_P1.3mm_Open_TrianglePad1.0x1.5mm, B.Cu at (105.1, 99.9)
- added Q3: MMBT3904, Package_TO_SOT_SMD:SOT-23, F.Cu at (116.1, 108.5)
- added Q4: MMBT3904, Package_TO_SOT_SMD:SOT-23, F.Cu at (116.6, 114.3)
- C1, C11, C12, C15, C2, C3, C8, C9: footprint Capacitor_SMD:C_0603_1608Metric -> Capacitor_SMD:C_0402_1005Metric
- J3: footprint Connector_PinHeader_2.54mm:PinHeader_1x04_P2.54mm_Vertical -> Connector_JST:JST_PH_B3B-PH-K_1x03_P2.00mm_Vertical
- J4: footprint Connector_PinHeader_2.54mm:PinHeader_1x04_P2.54mm_Vertical -> Connector_JST:JST_PH_B4B-PH-K_1x04_P2.00mm_Vertical
- Q1: value BC847BS -> MMBT3904; footprint Package_TO_SOT_SMD:SOT-363_SC-70-6 -> Package_TO_SOT_SMD:SOT-23
- R1, R10, R11, R12, R13, R14, R15, R16, R18, R19, R2, R20, R21, R22, R23, R3, R4, R5, R6, R7, R8, R9: footprint Resistor_SMD:R_0603_1608Metric -> Resistor_SMD:R_0402_1005Metric
- R17: value N.M. -> DNP; footprint Resistor_SMD:R_0603_1608Metric -> Resistor_SMD:R_0402_1005Metric
- TP1, TP11, TP12, TP13, TP2, TP3, TP4, TP5, TP6, TP7, TP8: moved to B.Cu
- moved TP4 40.1 mm to (107.8, 94.5), turned to 180 degrees
- moved TP3 37.1 mm to (113.0, 93.2), turned to 180 degrees
- moved TP12 35.2 mm to (115.0, 93.2), turned to 180 degrees
- moved TP7 35.0 mm to (112.3, 96.4), turned to 180 degrees
- moved TP8 33.8 mm to (111.4, 101.0), turned to 180 degrees
- moved R23 32.0 mm to (108.6, 104.0), turned to 90 degrees
- moved TP11 31.7 mm to (117.0, 93.2), turned to 180 degrees
- moved TP6 31.0 mm to (115.8, 96.5), turned to 180 degrees
- moved TP13 28.4 mm to (115.8, 103.2), turned to 180 degrees
- moved TP2 28.2 mm to (115.8, 98.8), turned to 180 degrees
- moved R22 27.7 mm to (111.3, 106.1), turned to 180 degrees
- moved TP5 24.5 mm to (113.5, 101.0), turned to 180 degrees
- moved R21 21.8 mm to (117.6, 111.9)
- moved R20 20.6 mm to (117.6, 110.8), turned to 180 degrees
- moved TP1 14.8 mm to (115.8, 101.0), turned to 180 degrees
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Connections:
- J3 pad 3: unconnected-(J3-Pin_3-Pad3) -> GND
- Q1 pad 1: GND -> Net-(Q1-B)
- Q1 pad 2: Net-(Q1A-B1) -> GND
- Q1 pad 3: Net-(Q1B-C2) -> Net-(Q1-C)
- R10 pad 2: Net-(Q1A-B1) -> Net-(Q1-B)
- R11 pad 2: Net-(Q1B-B2) -> Net-(Q3-B)
- R12 pad 2: Net-(Q1A-C1) -> Net-(Q1-C)
- R13 pad 2: Net-(Q1B-C2) -> Net-(Q3-C)
Routing:
- net GND: track 9.36 -> 47.7 mm, vias 62 -> 31
- net /RADIO-SPK: track 2.01 -> 24.0 mm, vias 0 -> 3
- net Net-(J3-Pin_2): track 0.00 -> 17.0 mm, vias 0 -> 3
- net /NRST: track 43.4 -> 26.5 mm, vias 2 -> 1
- net /817_PTT: track 0.00 -> 15.6 mm, vias 0 -> 4
- net Net-(J3-Pin_1): track 0.00 -> 14.9 mm, vias 0 -> 1
- net /RADIO-RX-PTT1: track 37.3 -> 24.1 mm
- net /BOOT0: track 17.4 -> 4.92 mm
- net Net-(J4-Pin_3): track 0.00 -> 10.7 mm
- net /RADIO-MIC: track 2.93 -> 13.4 mm, vias 0 -> 1
- net /USB-DP: track 13.1 -> 21.6 mm, vias 3 -> 2
- net Net-(J1-CC2): track 8.97 -> 17.4 mm, vias 0 -> 2
- net /USB-DN: track 14.0 -> 22.2 mm, vias 3 -> 2
- net /817_TX: track 0.00 -> 8.05 mm, vias 0 -> 2
- net /817_RX: track 0.00 -> 7.71 mm, vias 0 -> 2
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Other:
- board text removed: "3V3"
- board text removed: "BLD"
- board text removed: "GND"
- board text removed: "RST"
- board text removed: "SWC"
- board text removed: "SWO"

Commit message: Commit before assembly
Parts:
- added H10: Breakaway Hole, AIOC:breakawayHole, F.Cu at (86.5, 124.2)
- added H12: Breakaway Hole, AIOC:breakawayHole, F.Cu at (94.5, 124.2)
- added H13: Breakaway Hole, AIOC:breakawayHole, F.Cu at (93.0, 124.2)
- added H14: Breakaway Hole, AIOC:breakawayHole, F.Cu at (92.0, 124.2)
- added H15: Breakaway Hole, AIOC:breakawayHole, F.Cu at (100.2, 124.5)
- added H5: Breakaway Hole, AIOC:breakawayHole, F.Cu at (85.5, 124.2)
- added H6: Breakaway Hole, AIOC:breakawayHole, F.Cu at (91.0, 124.2)
- added H7: Breakaway Hole, AIOC:breakawayHole, F.Cu at (89.8, 124.2)
- added H8: Breakaway Hole, AIOC:breakawayHole, F.Cu at (87.5, 124.2)
- added H9: Breakaway Hole, AIOC:breakawayHole, F.Cu at (88.8, 124.2)
- H3, H4: footprint MountingHole:MountingHole_3.2mm_M3_ISO14580_Pad -> MountingHole:MountingHole_2.2mm_M2_ISO14580_Pad_TopBottom
- moved REF** 36.1 mm to (91.8, 118.2)
- moved R6 24.8 mm to (98.7, 100.2), turned to 90 degrees
- moved H3 24.5 mm to (100.8, 97.2)
- moved R7 24.1 mm to (98.7, 102.2), turned to -90 degrees
- moved J3 23.7 mm to (91.8, 131.2)
- moved R5 23.4 mm to (100.0, 104.3)
- moved TP11 23.3 mm to (97.5, 106.0)
- moved H4 23.2 mm to (86.8, 131.2)
- moved R20 23.1 mm to (98.3, 123.5)
- moved R21 23.1 mm to (98.3, 124.7)
- moved C11 23.1 mm to (100.0, 105.3)
- moved Q4 23.0 mm to (97.5, 127.0)
- moved R18 23.0 mm to (96.5, 123.5)
- moved R19 23.0 mm to (96.5, 124.7)
- moved J4 22.8 mm to (93.0, 126.2)
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Connections:
- R22 pad 1: Net-(J3-Pin_1) -> Net-(J3-Pin_2)
- R23 pad 1: Net-(J3-Pin_2) -> Net-(J3-Pin_1)
Routing:
- net GND: track 47.7 -> 24.9 mm, vias 31 -> 56
- net /RADIO-RX-PTT1: track 24.1 -> 17.4 mm, vias 2 -> 3
- net Net-(J1-CC1): track 10.1 -> 5.87 mm, vias 2 -> 0
- net /RADIO-TX: track 19.1 -> 15.5 mm
- net Net-(J3-Pin_1): track 14.9 -> 17.8 mm
- net /AFIN: track 10.5 -> 8.88 mm
- net /VIN: track 11.5 -> 13.0 mm
- net Net-(J1-CC2): track 17.4 -> 18.8 mm, vias 2 -> 0
- net Net-(U2-PB14): track 5.88 -> 4.48 mm
- net Net-(J3-Pin_2): track 17.0 -> 15.8 mm, vias 3 -> 1
- net /817_PTT: track 15.6 -> 14.5 mm, vias 4 -> 2
- net /RADIO-VP-PTT2: track 8.39 -> 7.49 mm, vias 2 -> 0
- net +3V3: track 53.5 -> 52.8 mm
- net Net-(U2-PA8): track 2.04 -> 1.34 mm
- net /RADIO-SPK: track 24.0 -> 23.4 mm, vias 3 -> 2
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- added copper zone on In2.Cu, net GND
Other:
- board size 21 x 31.5 mm -> 21 x 41.5 mm
- board text added: "AIOC V1.2"
- board text added: "AUD AUD PTT GND OUT IN OUT"
- board text added: "GND D+ D- +5"
- board text added: "GND SER SER OUT IN"
- board text added: "S. Kueppers AB1TJ"
- board text removed: "AIOC V1.0"
- board text removed: "S. Kueppers"
- board text removed: "SWD"
